Commit message: Update

File: urdf/riptide_actuators.urdf.xacro (robot description, xacro)
@@ -7,5 +7,5 @@
             <param name="baud_rate">115200</param>
         </hardware>
-		<joint name="thruster">
+		<joint name="$(arg prefix)_thruster">
             <command_interface name="position">
                 <param name="min">-1</param>
@@ -15,5 +15,5 @@
             <state_interface name="position"/>
         </joint>
-        <joint name="d_fin">
+        <joint name="$(arg prefix)_d_fin">
             <command_interface name="position">
                 <param name="min">"${-pi/2}"</param>
@@ -22,5 +22,5 @@
             <state_interface name="position"/>
         </joint>
-        <joint name="p_fin">
+        <joint name="$(arg prefix)_p_fin">
             <command_interface name="position">
                 <param name="min">"${-pi/2}"</param>
@@ -29,5 +29,5 @@
             <state_interface name="position"/>
         </joint>
-        <joint name="s_fin">
+        <joint name="$(arg prefix)_s_fin">
             <command_interface name="position">
                 <param name="min">"${-pi/2}"</param>
