Commit message: Fixing include

File: urdf/riptide.urdf.xacro (robot description, xacro)
@@ -1,5 +1,4 @@
 <?xml version="1.0"?>
 <robot name="$(arg prefix)" xmlns:xacro="http://www.ros.org/wiki/xacro">
-    <xacro:include filename="$(find riptide_description)/urdf/riptide.urdf.xacro"/>
     <!-- Rigid body description of the base link -->
 	<link name="$(arg prefix)">
@@ -55,3 +54,39 @@
         </sensor>
     </ros2_control>
+	<ros2_control name="riptide_actuators" type="system">
+        <hardware>
+            <plugin>riptide_hardware/ActuatorsHardware</plugin>
+            <param name="port">/dev/POLOLU</param>
+            <param name="baud_rate">115200</param>
+        </hardware>
+		<joint name="thruster">
+            <command_interface name="position">
+                <param name="min">-1</param>
+                <param name="max">1</param>
+            </command_interface>
+            <!-- <state_interface name="position"/> -->
+            <state_interface name="position"/>
+        </joint>
+        <joint name="d_fin">
+            <command_interface name="position">
+                <param name="min">"${-pi/2}"</param>
+                <param name="max">"${pi/2}"</param>
+            </command_interface>
+            <state_interface name="position"/>
+        </joint>
+        <joint name="p_fin">
+            <command_interface name="position">
+                <param name="min">"${-pi/2}"</param>
+                <param name="max">"${pi/2}"</param>
+            </command_interface>
+            <state_interface name="position"/>
+        </joint>
+        <joint name="s_fin">
+            <command_interface name="position">
+                <param name="min">"${-pi/2}"</param>
+                <param name="max">"${pi/2}"</param>
+            </command_interface>
+            <state_interface name="position"/>
+        </joint>
+    </ros2_control>
 </robot>

Commit message: Update

File: urdf/riptide.urdf.xacro (robot description, xacro)
@@ -35,58 +35,5 @@
 	<xacro:riptide_fin name="s" orientation="2"/>
     <!-- ROS2 control -->
-    <ros2_control name="riptide_imu" type="sensor">
-        <hardware>
-            <plugin>riptide_hardware/SpartonAHRSM1Hardware</plugin>
-            <param name="port">/dev/ttyUSB0</param>
-            <param name="baud_rate">115200</param>
-        </hardware>
-        <sensor name="imu">
-            <state_interface name="linear_acceleration.x"/>
-            <state_interface name="linear_acceleration.y"/>
-            <state_interface name="linear_acceleration.z"/>
-            <state_interface name="angular_velocity.x"/>
-            <state_interface name="angular_velocity.y"/>
-            <state_interface name="angular_velocity.z"/>
-            <state_interface name="orientation.x"/>
-            <state_interface name="orientation.y"/>
-            <state_interface name="orientation.z"/>
-            <state_interface name="orientation.w"/>
-        </sensor>
-    </ros2_control>
-	<ros2_control name="riptide_actuators" type="system">
-        <hardware>
-            <plugin>riptide_hardware/ActuatorsHardware</plugin>
-            <param name="port">/dev/POLOLU</param>
-            <param name="baud_rate">115200</param>
-        </hardware>
-		<joint name="thruster">
-            <command_interface name="position">
-                <param name="min">-1</param>
-                <param name="max">1</param>
-            </command_interface>
-            <!-- <state_interface name="position"/> -->
-            <state_interface name="position"/>
-        </joint>
-        <joint name="d_fin">
-            <command_interface name="position">
-                <param name="min">"${-pi/2}"</param>
-                <param name="max">"${pi/2}"</param>
-            </command_interface>
-            <state_interface name="position"/>
-        </joint>
-        <joint name="p_fin">
-            <command_interface name="position">
-                <param name="min">"${-pi/2}"</param>
-                <param name="max">"${pi/2}"</param>
-            </command_interface>
-            <state_interface name="position"/>
-        </joint>
-        <joint name="s_fin">
-            <command_interface name="position">
-                <param name="min">"${-pi/2}"</param>
-                <param name="max">"${pi/2}"</param>
-            </command_interface>
-            <state_interface name="position"/>
-        </joint>
-    </ros2_control>
+	<xacro:include filename="riptide_imu.urdf.xacro"/>
+	<xacro:include filename="riptide_actuators.urdf.xacro"/>
 </robot>

Commit message: Update

File: urdf/riptide.urdf.xacro (robot description, xacro)
@@ -24,5 +24,5 @@
 		</visual>
 	</link>
-	<joint name="$(arg prefix)_thruster" type="continuous">
+	<joint name="$(arg prefix)_thruster_joint" type="continuous">
 		<axis xyz="1 0 0"/>
 		<origin rpy="0 0 0" xyz="-0.51 0 0"/>

File: urdf/riptide_fin.urdf.xacro (robot description, xacro)
@@ -11,5 +11,5 @@
 			</visual>
 		</link>
-		<joint name="$(arg prefix)_${name}_fin" type="revolute">
+		<joint name="$(arg prefix)_${name}_joint" type="revolute">
 			<axis xyz="0 0 1"/>
 			<limit effort="1000.0" lower="${-pi/4}" upper="${pi/4}" velocity="0.5"/>
