Commit message: Update

File: urdf/riptide_tail.urdf.xacro (robot description, xacro)
@@ -9,5 +9,5 @@
             <param name="threshold_fin_commands">20</param>
         </hardware>
-		<joint name="$(arg prefix)_thruster">
+		<joint name="$(arg prefix)_thruster_joint">
             <command_interface name="velocity">
                 <param name="min">-1</param>
@@ -17,5 +17,5 @@
             <state_interface name="velocity"/>
         </joint>
-        <joint name="$(arg prefix)_d_fin">
+        <joint name="$(arg prefix)_d_joint">
             <command_interface name="position">
                 <param name="min">${-pi/4}</param>
@@ -26,5 +26,5 @@
             </state_interface>
         </joint>
-        <joint name="$(arg prefix)_p_fin">
+        <joint name="$(arg prefix)_p_joint">
             <command_interface name="position">
                 <param name="min">${-pi/4}</param>
@@ -34,5 +34,5 @@
             <state_interface name="position"/>
         </joint>
-        <joint name="$(arg prefix)_s_fin">
+        <joint name="$(arg prefix)_s_joint">
             <command_interface name="position">
                 <param name="min">${-pi/4}</param>
